Commit message: Added base URDF filesfor N3 and A3

File: swarmviz_description/urdf/a3.xacro (robot description, xacro)
@@ -1,4 +1,4 @@
 <?xml version="1.0"?>
-<robot name="m100"  xmlns:xacro="http://ros.org/wiki/xacro">
+<robot name="a3"  xmlns:xacro="http://ros.org/wiki/xacro">
 <!-- Properties -->
 <xacro:property name="namespace" value="$(arg namespace)" />
@@ -26,7 +26,7 @@
   <xacro:property name="rotor_drag_coefficient" value="8.06428e-05" />
   <xacro:property name="rolling_moment_coefficient" value="0.000001" />
-  <xacro:property name="origin_x" value="0" />
+  <xacro:property name="origin_x" value="7" />
   <xacro:property name="origin_y" value="0" />
-  <xacro:property name="origin_z" value="0.0" />
+  <xacro:property name="origin_z" value="0" />
   <!-- Property Blocks -->
 <xacro:property name = "body_inertia">

File: swarmviz_description/urdf/a3_base.xacro (robot description, xacro)
@@ -1,4 +1,4 @@
 <?xml version="1.0"?>
-<robot name="m100" xmlns:xacro="http://ros.org/wiki/xacro">
+<robot name="a3" xmlns:xacro="http://ros.org/wiki/xacro">
   <!-- Instantiate drone  "mechanics" -->
   <xacro:include filename="$(find swarmviz_description)/urdf/m100.xacro" />

File: swarmviz_description/urdf/multirotor_base.xacro (robot description, xacro)
@@ -36,5 +36,5 @@
     <link name="${robot_namespace}/base_link"></link>
     <joint name="${robot_namespace}/base_joint" type="fixed">
-      <origin xyz="0 0 0" rpy="0 0 0" />
+      <origin xyz="${origin_x} ${origin_y} ${origin_z}" rpy="0 0 0" />
       <parent link="${robot_namespace}/base_link" />
       <child link="${robot_namespace}/base_link_inertia" />
@@ -43,9 +43,9 @@
       <inertial>
         <mass value="${mass}" />  <!-- [kg] -->
-        <origin xyz="0 0 0" />
+        <origin xyz="${origin_x} ${origin_y} ${origin_z}" />
         <xacro:insert_block name="inertia" />
       </inertial>
       <visual>
-        <origin xyz="0 0 0" rpy="0 0 0" />
+        <origin xyz="${origin_x} ${origin_y} ${origin_z}" rpy="0 0 0" />
         <geometry>
           <xacro:if value="${use_mesh_file}">
@@ -58,5 +58,5 @@
       </visual>
       <collision>
-        <origin xyz="0 0 0" rpy="0 0 0" />
+       <origin xyz="${origin_x} ${origin_y} ${origin_z}" rpy="0 0 0" />
         <geometry>
           <box size="${body_width} ${body_width} ${body_height}" /> <!-- [m] [m] [m] -->
@@ -97,5 +97,5 @@
           </xacro:if>
           <xacro:unless value="${use_own_mesh}">
-            <mesh filename="package://m100_description/meshes/propeller_${direction}.dae"
+            <mesh filename="package://swarmviz_description/meshes/propeller_${direction}.dae"
               scale="${radius_rotor} ${radius_rotor} ${radius_rotor}" /> <!-- The propeller meshes have a radius of 1m -->
             <!-- <box size="${2*radius_rotor} 0.01 0.005"/> -->

File: swarmviz_description/urdf/n3.xacro (robot description, xacro)
@@ -1,4 +1,4 @@
 <?xml version="1.0"?>
-<robot name="m100"  xmlns:xacro="http://ros.org/wiki/xacro">
+<robot name="n3"  xmlns:xacro="http://ros.org/wiki/xacro">
 <!-- Properties -->
 <xacro:property name="namespace" value="$(arg namespace)" />

File: swarmviz_description/urdf/n3_base.xacro (robot description, xacro)
@@ -1,4 +1,4 @@
 <?xml version="1.0"?>
-<robot name="m100" xmlns:xacro="http://ros.org/wiki/xacro">
+<robot name="n3" xmlns:xacro="http://ros.org/wiki/xacro">
   <!-- Instantiate drone  "mechanics" -->
   <xacro:include filename="$(find swarmviz_description)/urdf/m100.xacro" />
